Commit message: auto gantry sampling

File: scripts/test_generator/rfl_description/urdf/rfl.urdf (robot description, URDF)
Before this commit: robot rfl, 44 links, 43 joints
Links:
- link bridge1: geometry collision mesh filename=D:/code_ws/pb_ws/compas_fab_pychoreo/scripts/test_generator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; visual mesh filename=D:/code_ws/pb_ws/compas_fab_pychoreo/scripts/test_generator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
- link bridge2: geometry collision mesh filename=D:/code_ws/pb_ws/compas_fab_pychoreo/scripts/test_generator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; visual mesh filename=D:/code_ws/pb_ws/compas_fab_pychoreo/scripts/test_generator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
- link robot11_base: geometry collision mesh filename=D:/code_ws/pb_ws/compas_fab_pychoreo/scripts/test_generator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; visual mesh filename=D:/code_ws/pb_ws/compas_fab_pychoreo/scripts/test_generator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
- link robot11_base_link: geometry collision mesh filename=D:/code_ws/pb_ws/compas_fab_pychoreo/scripts/test_generator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; visual mesh filename=D:/code_ws/pb_ws/compas_fab_pychoreo/scripts/test_generator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
- link robot11_link_1: geometry collision mesh filename=D:/code_ws/pb_ws/compas_fab_pychoreo/scripts/test_generator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; visual mesh filename=D:/code_ws/pb_ws/compas_fab_pychoreo/scripts/test_generator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
- link robot11_link_2: geometry collision mesh filename=D:/code_ws/pb_ws/compas_fab_pychoreo/scripts/test_generator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; visual mesh filename=D:/code_ws/pb_ws/compas_fab_pychoreo/scripts/test_generator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
- link robot11_link_3: geometry collision mesh filename=D:/code_ws/pb_ws/compas_fab_pychoreo/scripts/test_generator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; visual mesh filename=D:/code_ws/pb_ws/compas_fab_pychoreo/scripts/test_generator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
- link robot11_link_4: geometry collision mesh filename=D:/code_ws/pb_ws/compas_fab_pychoreo/scripts/test_generator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; visual mesh filename=D:/code_ws/pb_ws/compas_fab_pychoreo/scripts/test_generator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
- link robot11_link_5: geometry collision mesh filename=D:/code_ws/pb_ws/compas_fab_pychoreo/scripts/test_generator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; visual mesh filename=D:/code_ws/pb_ws/compas_fab_pychoreo/scripts/test_generator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
- link robot11_link_6: geometry collision mesh filename=D:/code_ws/pb_ws/compas_fab_pychoreo/scripts/test_generator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; visual mesh filename=D:/code_ws/pb_ws/compas_fab_pychoreo/scripts/test_generator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
- link robot11_xy_cart: geometry collision mesh filename=D:/code_ws/pb_ws/compas_fab_pychoreo/scripts/test_generator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; visual mesh filename=D:/code_ws/pb_ws/compas_fab_pychoreo/scripts/test_generator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
- link robot12_base: geometry collision mesh filename=D:/code_ws/pb_ws/compas_fab_pychoreo/scripts/test_generator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; visual mesh filename=D:/code_ws/pb_ws/compas_fab_pychoreo/scripts/test_generator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
- link robot12_base_link: geometry collision mesh filename=D:/code_ws/pb_ws/compas_fab_pychoreo/scripts/test_generator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; visual mesh filename=D:/code_ws/pb_ws/compas_fab_pychoreo/scripts/test_generator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
- link robot12_link_1: geometry collision mesh filename=D:/code_ws/pb_ws/compas_fab_pychoreo/scripts/test_generator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; visual mesh filename=D:/code_ws/pb_ws/compas_fab_pychoreo/scripts/test_generator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
- link robot12_link_2: geometry collision mesh filename=D:/code_ws/pb_ws/compas_fab_pychoreo/scripts/test_generator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; visual mesh filename=D:/code_ws/pb_ws/compas_fab_pychoreo/scripts/test_generator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
- link robot12_link_3: geometry collision mesh filename=D:/code_ws/pb_ws/compas_fab_pychoreo/scripts/test_generator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; visual mesh filename=D:/code_ws/pb_ws/compas_fab_pychoreo/scripts/test_generator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
- link robot12_link_4: geometry collision mesh filename=D:/code_ws/pb_ws/compas_fab_pychoreo/scripts/test_generator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; visual mesh filename=D:/code_ws/pb_ws/compas_fab_pychoreo/scripts/test_generator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
- link robot12_link_5: geometry collision mesh filename=D:/code_ws/pb_ws/compas_fab_pychoreo/scripts/test_generator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; visual mesh filename=D:/code_ws/pb_ws/compas_fab_pychoreo/scripts/test_generator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
- link robot12_link_6: geometry collision mesh filename=D:/code_ws/pb_ws/compas_fab_pychoreo/scripts/test_generator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; visual mesh filename=D:/code_ws/pb_ws/compas_fab_pychoreo/scripts/test_generator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
- link robot12_xy_cart: geometry collision mesh filename=D:/code_ws/pb_ws/compas_fab_pychoreo/scripts/test_generator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; visual mesh filename=D:/code_ws/pb_ws/compas_fab_pychoreo/scripts/test_generator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
- link robot21_base: geometry collision mesh filename=D:/code_ws/pb_ws/compas_fab_pychoreo/scripts/test_generator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; visual mesh filename=D:/code_ws/pb_ws/compas_fab_pychoreo/scripts/test_generator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
- link robot21_base_link: geometry collision mesh filename=D:/code_ws/pb_ws/compas_fab_pychoreo/scripts/test_generator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; visual mesh filename=D:/code_ws/pb_ws/compas_fab_pychoreo/scripts/test_generator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
- link robot21_link_1: geometry collision mesh filename=D:/code_ws/pb_ws/compas_fab_pychoreo/scripts/test_generator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; visual mesh filename=D:/code_ws/pb_ws/compas_fab_pychoreo/scripts/test_generator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
- link robot21_link_2: geometry collision mesh filename=D:/code_ws/pb_ws/compas_fab_pychoreo/scripts/test_generator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; visual mesh filename=D:/code_ws/pb_ws/compas_fab_pychoreo/scripts/test_generator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
- link robot21_link_3: geometry collision mesh filename=D:/code_ws/pb_ws/compas_fab_pychoreo/scripts/test_generator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; visual mesh filename=D:/code_ws/pb_ws/compas_fab_pychoreo/scripts/test_generator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
- link robot21_link_4: geometry collision mesh filename=D:/code_ws/pb_ws/compas_fab_pychoreo/scripts/test_generator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; visual mesh filename=D:/code_ws/pb_ws/compas_fab_pychoreo/scripts/test_generator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
- link robot21_link_5: geometry collision mesh filename=D:/code_ws/pb_ws/compas_fab_pychoreo/scripts/test_generator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; visual mesh filename=D:/code_ws/pb_ws/compas_fab_pychoreo/scripts/test_generator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
- link robot21_link_6: geometry collision mesh filename=D:/code_ws/pb_ws/compas_fab_pychoreo/scripts/test_generator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; visual mesh filename=D:/code_ws/pb_ws/compas_fab_pychoreo/scripts/test_generator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
- link robot21_xy_cart: geometry collision mesh filename=D:/code_ws/pb_ws/compas_fab_pychoreo/scripts/test_generator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; visual mesh filename=D:/code_ws/pb_ws/compas_fab_pychoreo/scripts/test_generator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
- link robot22_base: geometry collision mesh filename=D:/code_ws/pb_ws/compas_fab_pychoreo/scripts/test_generator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; visual mesh filename=D:/code_ws/pb_ws/compas_fab_pychoreo/scripts/test_generator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
- link robot22_base_link: geometry collision mesh filename=D:/code_ws/pb_ws/compas_fab_pychoreo/scripts/test_generator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; visual mesh filename=D:/code_ws/pb_ws/compas_fab_pychoreo/scripts/test_generator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
- link robot22_link_1: geometry collision mesh filename=D:/code_ws/pb_ws/compas_fab_pychoreo/scripts/test_generator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; visual mesh filename=D:/code_ws/pb_ws/compas_fab_pychoreo/scripts/test_generator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
- link robot22_link_2: geometry collision mesh filename=D:/code_ws/pb_ws/compas_fab_pychoreo/scripts/test_generator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; visual mesh filename=D:/code_ws/pb_ws/compas_fab_pychoreo/scripts/test_generator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
- link robot22_link_3: geometry collision mesh filename=D:/code_ws/pb_ws/compas_fab_pychoreo/scripts/test_generator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; visual mesh filename=D:/code_ws/pb_ws/compas_fab_pychoreo/scripts/test_generator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
- link robot22_link_4: geometry collision mesh filename=D:/code_ws/pb_ws/compas_fab_pychoreo/scripts/test_generator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; visual mesh filename=D:/code_ws/pb_ws/compas_fab_pychoreo/scripts/test_generator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
- link robot22_link_5: geometry collision mesh filename=D:/code_ws/pb_ws/compas_fab_pychoreo/scripts/test_generator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; visual mesh filename=D:/code_ws/pb_ws/compas_fab_pychoreo/scripts/test_generator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
- link robot22_link_6: geometry collision mesh filename=D:/code_ws/pb_ws/compas_fab_pychoreo/scripts/test_generator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; visual mesh filename=D:/code_ws/pb_ws/compas_fab_pychoreo/scripts/test_generator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
- link robot22_xy_cart: geometry collision mesh filename=D:/code_ws/pb_ws/compas_fab_pychoreo/scripts/test_generator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; visual mesh filename=D:/code_ws/pb_ws/compas_fab_pychoreo/scripts/test_generator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
- link world: geometry collision mesh filename=D:/code_ws/pb_ws/compas_fab_pychoreo/scripts/test_generator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; visual mesh filename=D:/code_ws/pb_ws/compas_fab_pychoreo/scripts/test_generator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
- link x_rail: geometry collision mesh filename=D:/code_ws/pb_ws/compas_fab_pychoreo/scripts/test_generator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; visual mesh filename=D:/code_ws/pb_ws/compas_fab_pychoreo/scripts/test_generator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
