Commit message: [WIP, #3] sweeping rays collision

File: tests/data/TC3_Igus/urdf/TC3_Igus.urdf (robot description, URDF)
Before this commit: robot TC3_Igus, 1 links, 0 joints
Links:
- link toolchanger_base: geometry collision mesh filename=package://TC3_Igus/meshes/collision/L0_collision_0.stl scale=0.001 0.001 0.001; collision mesh filename=package://TC3_Igus/meshes/collision/L0_collision_1.stl scale=0.001 0.001 0.001

File: tests/data/g1/urdf/g1.urdf (robot description, URDF)
Before this commit: robot g1, 3 links, 2 joints
Joints:
- joint joint_gripper_jaw_l: origin xyz=0.0 0.0 0.0 rpy=0.0 -0.0 0.0 -> xyz=0.0 0.0 0.0 rpy=0.0 0.0 0.0
- joint joint_gripper_jaw_r: axis -1.0 0.0 0.0 -> -1.0 -0.0 -0.0; origin xyz=0.0 0.0 0.0 rpy=0.0 -0.0 0.0 -> xyz=0.0 0.0 0.0 rpy=0.0 0.0 0.0
